Commit message: feat: update robot colors

File: P2 Go Chase It/my_robot/urdf/my_robot.xacro (robot description, xacro)
@@ -8,4 +8,7 @@
     <color rgba="1.0 0.0 0.0 1.0"/>
   </material>
+  <material name="yellow">
+    <color rgba="1.0 1.0 0.0 1.0"/>
+  </material>
   <link name="robot_footprint"></link>
   <joint name="robot_footprint_joint" type="fixed">
@@ -62,9 +65,9 @@
         <cylinder radius="0.15" length="0.1"/>
       </geometry>
-      <material name="green"/>
+      <material name="red"/>
     </visual>
   </link>
   <gazebo reference="right_wheel">
-    <material>Gazebo/Green</material>
+    <material>Gazebo/Red</material>
   </gazebo>
   <link name='chassis'>
@@ -90,5 +93,5 @@
         <box size=".4 .2 .15"/>
       </geometry>
-      <material name="red"/>
+      <material name="yellow"/>
     </visual>
     <collision name='back_caster_collision'>
@@ -120,5 +123,5 @@
   </link>
   <gazebo reference="chassis">
-    <material>Gazebo/Red</material>
+    <material>Gazebo/Yellow</material>
   </gazebo>
   <joint type="continuous" name="left_wheel_hinge">
@@ -151,11 +154,11 @@
       <origin xyz="0 0 0" rpy="0 0 0"/>
       <geometry>
-	<box size="0.05 0.05 0.05"/>
-      </geometry>
-    </collision>
-    <visual>
-      <origin xyz="0 0 0" rpy="0 0 0"/>
-      <geometry>
-	<box size="0.05 0.05 0.05"/>
+        <box size="0.05 0.05 0.05"/>
+      </geometry>
+    </collision>
+    <visual>
+      <origin xyz="0 0 0" rpy="0 0 0"/>
+      <geometry>
+        <box size="0.05 0.05 0.05"/>
       </geometry>
     </visual>
@@ -180,11 +183,11 @@
       <origin xyz="0 0 0" rpy="0 0 0"/>
       <geometry>
-	<box size="0.1 0.1 0.1"/>
-      </geometry>
-    </collision>
-    <visual>
-      <origin xyz="0 0 0" rpy="0 0 0"/>
-      <geometry>
-	<mesh filename="package://my_robot/meshes/hokuyo.dae"/>
+        <box size="0.1 0.1 0.1"/>
+      </geometry>
+    </collision>
+    <visual>
+      <origin xyz="0 0 0" rpy="0 0 0"/>
+      <geometry>
+        <mesh filename="package://my_robot/meshes/hokuyo.dae"/>
       </geometry>
     </visual>
